File: hardware/kikad/pcb.kicad_sch (KiCad schematic)
At the start: 22 parts, among them J1 Output

Commit message: Revert "make the v0.3 read to use"
This reverts commit 2651ca28fcff3cfeeb4fb146a67662ef7f719936.
Parts:
- removed BZ1: Buzzer, Buzzer_Beeper:MagneticBuzzer_ProSignal_ABI-010-RC, symbol Device:Buzzer
- removed J1: Output, Connector_JST:JST_XH_B3B-XH-A_1x03_P2.50mm_Vertical, symbol Connector:Conn_01x03_Pin
- removed U2: ~, esp_32_c3_supper_mini:PN532 NFC RFID, symbol esp_c3_32_supper_mini:PN532_NFC_RFID_module_V3
- added D7: LED_Dual_AKA, Connector_JST:JST_XH_B3B-XH-A_1x03_P2.50mm_Vertical, symbol Device:LED_Dual_AKA
- added J2: BOARD, Connector_PinSocket_2.54mm:PinSocket_1x02_P2.54mm_Vertical, symbol Connector:Conn_01x02_Pin
- R14: value 0 -> 150
Connections:
- net B: now also U1.7 (GPIO1); no longer U1.16 (GPIO21)
- net G: now also U1.6 (GPIO2); no longer U1.15 (GPIO20)
- net GND: now also D7.2 (K), J2.2 (Pin_2)
- net R: now also U1.5 (GPIO3); no longer U1.14 (GPIO10)
- net at U1.9 (GPIO5): now also R14.1
- net at U1.10 (GPIO6): now also R13.2
- net at R13.1: now also D7.3 (A2); no longer U1.13 (GPIO9/SCL)
- net at U1.1 (5V): now also J2.1 (Pin_1)
- net at R14.2: now also D7.1 (A1); no longer U1.3 (3V3)
- no-connect marks 8 -> 10
Other:
- moved on the sheet: D1, D2, D3, D4, R1, R10, R11, R12, R2, R3, R4, R5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
