File: hardware/main/_autosave-pcb.kicad_pcb (KiCad board)
At the start: 2 copper layers, 55 x 55 mm, 24 parts, among them J1 Conn_01x02_Socket, J2 Conn_01x02_Socket

Commit message: update the PCB and test stand project folder
Parts:
- moved BZ1 1.45 mm to (109.4, 82.0)
Routing:
- net Net-(BZ1-+): track 16.6 -> 17.2 mm
Changed lines of the file:
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@@
 			(at 0 -0.5 90)
 			(unlocked yes)
-			(layer "F.SilkS")
+			(layer "B.SilkS")
 			(hide yes)
 			(effects
@@
 					(thickness 0.1)
 				)
+				(justify mirror)
 			)
 		)
@@
 	(footprint "Buzzer_Beeper:MagneticBuzzer_ProSignal_ABI-010-RC"
 		(layer "F.Cu")
-		(at 110.85 82)
+		(at 109.4 82)
 		(descr "Buzzer, Elektromagnetic Beeper, Summer, 12V-DC,")
 		(tags "Pro Signal ABI-010-RC ")
@@
 	)
 	(segment
-		(start 108 65.61)
-		(end 108 88.9)
+		(start 107.2 89.7)
+		(end 105.2 91.7)
+		(width 0.8)
+		(layer "B.Cu")
+		(net 10)
+	)
+	(segment
+		(start 107.501 66.580263)
+		(end 107.202 66.879263)
+		(width 0.8)
+		(layer "B.Cu")
+		(net 10)
+	)
+	(segment
+		(start 107.202 85.133419)
+		(end 107.2 85.135419)
 		(width 0.8)
 		(layer "B.Cu")
@@
 	)
 	(segment
-		(start 108 88.9)
-		(end 105.2 91.7)
+		(start 108 65.61)
+		(end 107.501 66.109)
+		(width 0.8)
+		(layer "B.Cu")
+		(net 10)
+	)
+	(segment
+		(start 107.501 66.109)
+		(end 107.501 66.580263)
+		(width 0.8)
+		(layer "B.Cu")
+		(net 10)
+	)
+	(segment
+		(start 107.2 85.135419)
+		(end 107.2 89.7)
+		(width 0.8)
+		(layer "B.Cu")
+		(net 10)
+	)
+	(segment
+		(start 107.202 66.879263)
+		(end 107.202 85.133419)
 		(width 0.8)
 		(layer "B.Cu")
@@
 	(segment
 		(start 111.4 65.61)
-		(end 111.4 81.45)
+		(end 111.4 80)
 		(width 0.8)
 		(layer "B.Cu")
@@
 	)
 	(segment
-		(start 111.4 81.45)
-		(end 110.85 82)
-		(width 0.8)
-		(layer "B.Cu")
+		(start 111.4 80)
+		(end 109.4 82)
+		(width 0.8)
+		(layer "B.Cu")
