File: hardware/main/pcb.kicad_pcb (KiCad board)
At the start: 2 copper layers, 55 x 55 mm, 29 parts, among them J3 Conn_01x03_Socket, Q1 BC547, Q2 BC547, Q3 BC547, U1 ESP32 C3 supper mini

Commit message: update the media
Parts:
- moved BZ1 5.23 mm to (115.1, 85.0), turned to -90 degrees
- moved R13 3.43 mm to (123.9, 81.5), turned to -90 degrees
- moved U1 2.84 mm to (129.8, 65.8)
- moved J3 0.90 mm to (134.2, 92.3)
Routing:
- net /G: track 10.3 -> 21.0 mm
- net /R: track 26.5 -> 31.7 mm
- net Net-(BZ1-+): track 6.49 -> 10.5 mm
- net Net-(J3-Pin_3): track 39.1 -> 42.1 mm
- net Net-(U1-GPIO7/SS): track 22.1 -> 24.5 mm
- net /B: track 6.10 -> 8.46 mm
- net +5V: track 70.4 -> 72.7 mm
- net Net-(U1-GPIO4/SCK): track 3.73 -> 4.91 mm
- net Net-(U1-GPIO2): track 3.73 -> 4.91 mm
- net Net-(U1-GPIO1): track 3.73 -> 4.91 mm
- net Net-(U1-GPIO3): track 3.73 -> 4.91 mm
- net Net-(U1-3V3): track 4.05 -> 4.91 mm
Other:
- board text added: "Kyiv, Ukraine HackerSpace NU31"
- board text added: "Prismo 1.0.0-alpha.2"
- board text removed: "Prismo 1.0.0-alpha.1 Kyiv, Ukraine HackerSpace NU31"

Commit message: prepare the rc
Other:
- board text added: "Prismo 1.0.0-RC.1"
- board text removed: "Prismo 1.0.0-alpha.2"
Changed lines of the file:
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@@
 		)
 	)
-	(gr_text "Prismo 1.0.0-alpha.2"
+	(gr_text "Prismo 1.0.0-RC.1"
 		(at 136.9 51.4 0)
 		(layer "B.SilkS")
