File: hardware/ac/pcb.kicad_sch (KiCad schematic)
At the start: 11 parts, among them J1 AC IN 100-240V, J2 AC OUT (switched L, N), J3 To main board, K1 SRD-05VDC-SL-C, Q1 2N7000, U1 HLK-5M05

Commit message: small updates
Other:
- note removed: "F1 limits the relay load (<=2A)"
