File: hardware/dcdc/pcb.kicad_sch (KiCad schematic)
At the start: 12 parts, among them J1 DC IN 7-40V, J2 LOAD 1=VIN 2=SW GND, J3 To main board, J4 BUTTON NO, Q2 IRLZ44N, U1 LM2596HV-5.0

Commit message: small updates
Parts:
- J1: value DC IN 7-40V -> DC IN 7-36V
Other:
- note added: "PRISMO: DC-DC 7-36V power board"
- note removed: "PRISMO: DC-DC 7-40V power board"
Changed lines of the file:
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@@
 	(generator_version "10.0")
 	(paper "A4")
-	(text "PRISMO: DC-DC 7-40V power board"
+	(text "PRISMO: DC-DC 7-36V power board"
 		(exclude_from_sim no)
 		(at 25.4 38.1 0)
@@
 			)
 		)
-		(property "Value" "DC IN 7-40V"
+		(property "Value" "DC IN 7-36V"
 			(at 25.4 57.785 0)
 			(show_name no)
